File: hdi20-floppy.brd (EAGLE design)
At the start: 16.5 x 30.5 mm, 2 parts

Commit message: 20250725
Parts:
- moved E$1 10.2 mm to (2.84, 12.5)
- moved E$2 3.81 mm to (8.89, 15.2)
Routing:
- net S$10: track 14.8 -> 22.1 mm
- net S$7: track 9.14 -> 7.81 mm
- net S$8: track 9.36 -> 8.03 mm
- net S$6: track 8.91 -> 7.58 mm
- net S$5: track 8.69 -> 7.36 mm
- net S$3: track 8.24 -> 6.91 mm
- net S$4: track 8.47 -> 7.14 mm
- net S$2: track 8.11 -> 7.00 mm
- net S$1: track 8.33 -> 7.23 mm
- net S$9: track 9.60 -> 8.78 mm
Other:
- board size 16.5 x 30.5 mm -> 12.1 x 30.5 mm
- board text added: "< Teal & orange wires"
- board text added: "HDI-20 Floppy Adapter"
- board text added: "NOTE: 5V only!"
- board text removed: "Orange and teal wires this side"
